File: FAST/FAST Controller.kicad_pcb (KiCad board)
At the start: 2 copper layers, 125 x 50.8 mm, 67 parts, among them J1 APM_POWER_MODULE, J10 CH3_THROTTLE_ESC_BEC_IN, J11 CH4, J12 CH5, J13 CH6, J14 CH7, J15 CH8, J2 ESP_AIR_SD_MODULE, J3 M5STACK_IMU_PRO, J4 CRSF_RX, J5 OUTBOARD_UART, J6 RX_PWM_1_4, J7 RX_PWM_5_8, J8 CH1, J9 CH2, U1 FAST Teensy 4.0 DIP Carrier, U2 ESP_AIR / XIAO ESP32-S3, U3 CD74HCT157E_CH1_4, U4 CD74HCT157E_CH5_8, U5 ADM706ARZ

Commit message: Release FAST Controller V2.1 production corrections
Parts:
- added R30: 10k, R_0805_2012Metric_Pad1.20x1.40mm_HandSolder, F.Cu at (84.5, 29.8)
- turned D1 to 180 degrees
- turned D2 to 180 degrees
Connections:
- D1 pad 1: /+5V_PM_BEC -> /+5V_LOGIC
- D1 pad 2: /+5V_LOGIC -> /+5V_PM_BEC
- D2 pad 1: /+5V_ESC_BEC -> /+5V_LOGIC
- D2 pad 2: /+5V_LOGIC -> /+5V_ESC_BEC
Other:
- board text added: "FAST CONTROLLER V2.1"
- board text added: "FIT INSULATED LINK: J4-2 TO TP3"
- board text removed: "FAST CONTROLLER V2"
Changed lines of the file:
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@@
 	(footprint "D_SOD-128"
 		(layer "F.Cu")
-		(at 91.2 24)
+		(at 91.2 24 180)
 		(descr "D_SOD-128 (CFP5 SlimSMAW), https://assets.nexperia.com/documents/outline-drawing/SOD128.pdf")
 		(tags "D_SOD-128")
@@
 		(duplicate_pad_numbers_are_jumpers no)
 		(fp_line
-			(start -3.16 -1.36)
-			(end -3.16 1.36)
+			(start -3.16 1.36)
+			(end 1.9 1.36)
 			(stroke
 				(width 0.12)
@@
 		)
 		(fp_line
-			(start -3.16 1.36)
-			(end 1.9 1.36)
+			(start -3.16 -1.36)
+			(end -3.16 1.36)
 			(stroke
 				(width 0.12)
@@
 		)
 		(fp_line
-			(start -3.15 -1.5)
+			(start 3.15 1.5)
 			(end -3.15 1.5)
 			(stroke
@@
 		)
 		(fp_line
-			(start -3.15 -1.5)
-			(end 3.15 -1.5)
+			(start 3.15 -1.5)
+			(end 3.15 1.5)
 			(stroke
 				(width 0.05)
@@
 		)
 		(fp_line
-			(start 3.15 -1.5)
-			(end 3.15 1.5)
+			(start -3.15 -1.5)
+			(end 3.15 -1.5)
 			(stroke
 				(width 0.05)
@@
 		)
 		(fp_line
-			(start 3.15 1.5)
+			(start -3.15 -1.5)
 			(end -3.15 1.5)
 			(stroke
@@
 			(layers "F.Cu" "F.Mask" "F.Paste")
 			(roundrect_rratio 0.1785714286)
-			(net "/+5V_ESC_BEC")
+			(net "/+5V_LOGIC")
 		)
 		(pad "2" smd roundrect
@@
 			(layers "F.Cu" "F.Mask" "F.Paste")
 			(roundrect_rratio 0.1785714286)
-			(net "/+5V_LOGIC")
+			(net "/+5V_ESC_BEC")
 		)
 		(embedded_fonts no)
@@
 	(footprint "D_SOD-128"
 		(layer "F.Cu")
-		(at 91 66)
+		(at 91 66 180)
 		(descr "D_SOD-128 (CFP5 SlimSMAW), https://assets.nexperia.com/documents/outline-drawing/SOD128.pdf")
 		(tags "D_SOD-128")
@@
 		(duplicate_pad_numbers_are_jumpers no)
 		(fp_line
-			(start -3.16 -1.36)
-			(end -3.16 1.36)
+			(start -3.16 1.36)
+			(end 1.9 1.36)
 			(stroke
 				(width 0.12)
@@
 		)
 		(fp_line
-			(start -3.16 1.36)
-			(end 1.9 1.36)
+			(start -3.16 -1.36)
+			(end -3.16 1.36)
 			(stroke
 				(width 0.12)
@@
 		)
 		(fp_line
-			(start -3.15 -1.5)
+			(start 3.15 1.5)
 			(end -3.15 1.5)
 			(stroke
@@
 		)
 		(fp_line
-			(start -3.15 -1.5)
-			(end 3.15 -1.5)
+			(start 3.15 -1.5)
+			(end 3.15 1.5)
 			(stroke
 				(width 0.05)
@@
 		)
 		(fp_line
-			(start 3.15 -1.5)
-			(end 3.15 1.5)
+			(start -3.15 -1.5)
+			(end 3.15 -1.5)
 			(stroke
 				(width 0.05)
@@
 		)
 		(fp_line
-			(start 3.15 1.5)
+			(start -3.15 -1.5)
 			(end -3.15 1.5)
 			(stroke
@@
 			(layers "F.Cu" "F.Mask" "F.Paste")
 			(roundrect_rratio 0.1785714286)
-			(net "/+5V_PM_BEC")
+			(net "/+5V_LOGIC")
 		)
 		(pad "2" smd roundrect
@@
 			(layers "F.Cu" "F.Mask" "F.Paste")
 			(roundrect_rratio 0.1785714286)
-			(net "/+5V_LOGIC")
+			(net "/+5V_PM_BEC")
 		)
 		(embedded_fonts no)
@@
 	(footprint "R_0805_2012Metric_Pad1.20x1.40mm_HandSolder"
 		(layer "F.Cu")
+		(at 84.5 29.8498 -90)
+		(descr "Resistor SMD 0805 (2012 Metric), hand-solder pads")
+		(tags "resistor handsolder")
+		(property "Reference" "R30"
+			(at -3 0 90)
+			(layer "F.SilkS")
+			(effects
+				(font
+					(size 0.8 0.8)
+					(thickness 0.15)
+				)
+			)
+		)
+		(property "Value" "10k"
+			(at 3 0 90)
+			(layer "F.SilkS")
+			(effects
+				(font
+					(size 0.8 0.8)
+					(thickness 0.15)
+				)
+			)
+		)
+		(property "Datasheet" ""
+			(at 0 0 0)
+			(layer "F.Fab")
+			(hide yes)
+			(effects
+				(font
+					(size 1.27 1.27)
+				)
+			)
+		)
+		(property "Description" "MUX_SELECT fail-safe pull-down"
+			(at 0 0 0)
+			(layer "F.Fab")
+			(hide yes)
+			(effects
+				(font
+					(size 1.27 1.27)
+				)
+			)
+		)
+		(attr smd)
+		(duplicate_pad_numbers_are_jumpers no)
+		(fp_line
+			(start -0.227064 0.735)
+			(end 0.227064 0.735)
+			(stroke
+				(width 0.12)
+				(type solid)
+			)
+			(layer "F.SilkS")
+		)
+		(fp_line
+			(start -0.227064 -0.735)
+			(end 0.227064 -0.735)
+			(stroke
+				(width 0.12)
+				(type solid)
+			)
+			(layer "F.SilkS")
+		)
+		(fp_rect
+			(start -1.85 -0.95)
+			(end 1.85 0.95)
+			(stroke
+				(width 0.05)
+				(type solid)
+			)
+			(fill no)
+			(layer "F.CrtYd")
+		)
+		(pad "1" smd roundrect
+			(at -1 0)
+			(size 1.2 1.4)
+			(layers "F.Cu" "F.Mask" "F.Paste")
+			(roundrect_rratio 0.208333)
+			(net "/MUX_SELECT")
+		)
+		(pad "2" smd roundrect
+			(at 1 0)
+			(size 1.2 1.4)
+			(layers "F.Cu" "F.Mask" "F.Paste")
+			(roundrect_rratio 0.208333)
+			(net "/GND")
+		)
+		(embedded_fonts no)
+		(model "${KICAD10_3DMODEL_DIR}/Resistor_SMD.3dshapes/R_0805_2012Metric.step"
+			(offset
+				(xyz 0 0 0)
+			)
+			(scale
+				(xyz 1 1 1)
+			)
+			(rotate
+				(xyz 0 0 0)
+			)
+		)
+	)
+	(footprint "R_0805_2012Metric_Pad1.20x1.40mm_HandSolder"
+		(layer "F.Cu")
 		(at 130 25)
 		(descr "Resistor SMD 0805 (2012 Metric), square (rectangular) end terminal, IPC-7351 nominal with elongated pad for handsoldering. (Body size source: IPC-SM-782 page 72, https://www.pcb-3d.com/wordpress/wp-content/uploads/ipc-sm-782a_amendment_1_and_2.pdf)")
@@
 		)
 	)
-	(gr_text "FAST CONTROLLER V2"
+	(gr_text "FIT INSULATED LINK: J4-2 TO TP3"
+		(at 84 68.8 0)
+		(layer "B.SilkS")
+		(effects
+			(font
+				(size 0.8 0.8)
+				(thickness 0.12)
+			)
+			(justify mirror)
+		)
+	)
+	(gr_text "FAST CONTROLLER V2.1"
 		(at 60 35 0)
 		(layer "B.SilkS")

Commit message: Release FAST Controller V2.2 servo power correction
Connections:
- J10 pad 1: /+5V_ESC_BEC -> /GND
- J10 pad 2: /GND -> /+5V_ESC_BEC
- J11 pad 1: /+5V_ESC_BEC -> /GND
- J11 pad 2: /GND -> /+5V_ESC_BEC
- J12 pad 1: /+5V_ESC_BEC -> /GND
- J12 pad 2: /GND -> /+5V_ESC_BEC
- J13 pad 1: /+5V_ESC_BEC -> /GND
- J13 pad 2: /GND -> /+5V_ESC_BEC
- J14 pad 1: /+5V_ESC_BEC -> /GND
- J14 pad 2: /GND -> /+5V_ESC_BEC
- J15 pad 1: /+5V_ESC_BEC -> /GND
- J15 pad 2: /GND -> /+5V_ESC_BEC
- J8 pad 1: /+5V_ESC_BEC -> /GND
- J8 pad 2: /GND -> /+5V_ESC_BEC
- J9 pad 1: /+5V_ESC_BEC -> /GND
- J9 pad 2: /GND -> /+5V_ESC_BEC
Routing:
- net /+5V_ESC_BEC: track 175.4 -> 171.4 mm
Changed lines of the file:
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@@
 			(layers "*.Cu" "*.Mask")
 			(remove_unused_layers no)
-			(net "/+5V_ESC_BEC")
+			(net "/GND")
 		)
 		(pad "2" thru_hole circle
@@
 			(layers "*.Cu" "*.Mask")
 			(remove_unused_layers no)
-			(net "/GND")
+			(net "/+5V_ESC_BEC")
 		)
 		(pad "3" thru_hole circle
@@
 			(layers "*.Cu" "*.Mask")
 			(remove_unused_layers no)
-			(net "/+5V_ESC_BEC")
+			(net "/GND")
 		)
 		(pad "2" thru_hole circle
@@
 			(layers "*.Cu" "*.Mask")
 			(remove_unused_layers no)
-			(net "/GND")
+			(net "/+5V_ESC_BEC")
 		)
 		(pad "3" thru_hole circle
@@
 			(layers "*.Cu" "*.Mask")
 			(remove_unused_layers no)
-			(net "/+5V_ESC_BEC")
+			(net "/GND")
 		)
 		(pad "2" thru_hole circle
@@
 			(layers "*.Cu" "*.Mask")
 			(remove_unused_layers no)
-			(net "/GND")
+			(net "/+5V_ESC_BEC")
 		)
 		(pad "3" thru_hole circle
@@
 			(layers "*.Cu" "*.Mask")
 			(remove_unused_layers no)
-			(net "/+5V_ESC_BEC")
+			(net "/GND")
 		)
 		(pad "2" thru_hole circle
@@
 			(layers "*.Cu" "*.Mask")
 			(remove_unused_layers no)
-			(net "/GND")
+			(net "/+5V_ESC_BEC")
 		)
 		(pad "3" thru_hole circle
@@
 			(layers "*.Cu" "*.Mask")
 			(remove_unused_layers no)
-			(net "/+5V_ESC_BEC")
+			(net "/GND")
 		)
 		(pad "2" thru_hole circle
@@
 			(layers "*.Cu" "*.Mask")
 			(remove_unused_layers no)
-			(net "/GND")
+			(net "/+5V_ESC_BEC")
 		)
 		(pad "3" thru_hole circle
@@
 			(layers "*.Cu" "*.Mask")
 			(remove_unused_layers no)
-			(net "/+5V_ESC_BEC")
+			(net "/GND")
 		)
 		(pad "2" thru_hole circle
@@
 			(layers "*.Cu" "*.Mask")
 			(remove_unused_layers no)
-			(net "/GND")
+			(net "/+5V_ESC_BEC")
 		)
 		(pad "3" thru_hole circle
@@
 			(layers "*.Cu" "*.Mask")
 			(remove_unused_layers no)
-			(net "/+5V_ESC_BEC")
+			(net "/GND")
 		)
 		(pad "2" thru_hole circle
@@
 			(layers "*.Cu" "*.Mask")
 			(remove_unused_layers no)
-			(net "/GND")
+			(net "/+5V_ESC_BEC")
 		)
 		(pad "3" thru_hole circle
@@
 			(layers "*.Cu" "*.Mask")
 			(remove_unused_layers no)
-			(net "/+5V_ESC_BEC")
+			(net "/GND")
 		)
 		(pad "2" thru_hole circle
@@
 			(layers "*.Cu" "*.Mask")
 			(remove_unused_layers no)
-			(net "/GND")
+			(net "/+5V_ESC_BEC")
 		)
 		(pad "3" thru_hole circle
@@
 	)
 	(segment
-		(start 139.08 41)
-		(end 139.08 48)
+		(start 136.54 41)
+		(end 136.54 48)
 		(width 1)
 		(layer "B.Cu")
@@
 	)
 	(segment
-		(start 139.08 50)
-		(end 139.08 54)
+		(start 136.54 50)
+		(end 136.54 54)
 		(width 1)
 		(layer "B.Cu")
@@
 	)
 	(segment
-		(start 139.08 54)
-		(end 139.08 58)
+		(start 136.54 54)
+		(end 136.54 58)
 		(width 1)
 		(layer "B.Cu")
@@
 	)
 	(segment
-		(start 139.08 58)
-		(end 139.08 62)
+		(start 136.54 58)
+		(end 136.54 62)
 		(width 1)
 		(layer "B.Cu")
@@
 	)
 	(segment
-		(start 139.08 41)
-		(end 139.08 37)
+		(start 136.54 41)
+		(end 136.54 37)
 		(width 1)
 		(layer "B.Cu")
@@
 	)
 	(segment
-		(start 139.08 48)
+		(start 136.54 48)
 		(end 127.9017 48)
 		(width 1)
@@
 	)
 	(segment
-		(start 139.08 48)
-		(end 139.08 50)
+		(start 136.54 48)
+		(end 136.54 50)
 		(width 1)
 		(layer "B.Cu")
@@
 	)
 	(segment
-		(start 139.08 37)
-		(end 139.08 33)
+		(start 136.54 37)
+		(end 136.54 33)
 		(width 1)
 		(layer "B.Cu")
@@
 	)
 	(segment
-		(start 139.08 29)
-		(end 139.08 33)
+		(start 136.54 29)
+		(end 136.54 33)
 		(width 1)
 		(layer "B.Cu")
@@
 	(segment
 		(start 134.08 24)
-		(end 139.08 29)
+		(end 136.54 29)
 		(width 1)
 		(layer "B.Cu")

Commit message: Update FAST Controller V2.2 schematic and ground stitching
Routing:
- net /GND: track 26.8 -> 28.8 mm, vias 6 -> 9
- net /TEENSY_PWM7_RAW: track 61.9 -> 62.9 mm
Changed lines of the file:
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@@
 		)
+	)
+	(segment
+		(start 72.5 64)
+		(end 72.5 65)
+		(width 0.5)
+		(layer "F.Cu")
+		(net "/GND")
+	)
+	(segment
+		(start 72.5 65)
+		(end 73.5 65)
+		(width 0.5)
+		(layer "F.Cu")
+		(net "/GND")
 	)
 	(via
@@
 	(via
 		(at 130 68)
+		(size 0.8)
+		(drill 0.4)
+		(layers "F.Cu" "B.Cu")
+		(net "/GND")
+	)
+	(via
+		(at 60 56)
+		(size 0.8)
+		(drill 0.4)
+		(layers "F.Cu" "B.Cu")
+		(net "/GND")
+	)
+	(via
+		(at 72.5 65)
+		(size 0.8)
+		(drill 0.4)
+		(layers "F.Cu" "B.Cu")
+		(net "/GND")
+	)
+	(via
+		(at 73.5 65)
 		(size 0.8)
 		(drill 0.4)
@@
 	)
 	(segment
+		(start 76.3 66.4)
+		(end 77 65.4391)
+		(width 0.2)
+		(layer "F.Cu")
+		(net "/TEENSY_PWM7_RAW")
+	)
+	(segment
+		(start 69 65.4391)
+		(end 69.7 66.4)
+		(width 0.2)
+		(layer "F.Cu")
+		(net "/TEENSY_PWM7_RAW")
+	)
+	(segment
 		(start 82.4957 65.4391)
 		(end 83.3451 64.5897)
@@
 	)
 	(segment
+		(start 77 65.4391)
+		(end 82.4957 65.4391)
+		(width 0.2)
+		(layer "F.Cu")
+		(net "/TEENSY_PWM7_RAW")
+	)
+	(segment
 		(start 83.3451 64.5897)
 		(end 111.41 64.5897)
@@
 	)
 	(segment
+		(start 69.7 66.4)
+		(end 76.3 66.4)
+		(width 0.2)
+		(layer "F.Cu")
+		(net "/TEENSY_PWM7_RAW")
+	)
+	(segment
 		(start 53.8191 65.4391)
-		(end 82.4957 65.4391)
-		(width 0.2)
-		(layer "F.Cu")
+		(end 69 65.4391)
+		(width 0.2)
+		(layer "F.Cu")
