File: FAST/FAST Controller.kicad_sch (KiCad schematic)
At the start: 63 parts, among them J1 APM_POWER_MODULE, J10 CH3_THROTTLE_ESC_BEC_IN, J11 CH4, J12 CH5, J13 CH6, J14 CH7, J15 CH8, J2 ESP_AIR_SD_MODULE, J3 M5STACK_IMU_PRO, J4 CRSF_RX, J5 GPS_AIRSPEED_OUTBOARD_UART, J6 RX_PWM_1_4, J7 RX_PWM_5_8, J8 CH1, J9 CH2, U1 FAST Teensy 4.0 DIP Carrier, U2 ESP_AIR / XIAO ESP32-S3, U3 CD74HCT157E_CH1_4, U4 CD74HCT157E_CH5_8, U5 ADM706ARZ

Commit message: Release FAST Controller V2.1 production corrections
Parts:
- added R30: 10k, Resistor_SMD:R_0805_2012Metric_Pad1.20x1.40mm_HandSolder, symbol Device:R
Connections:
- net +5V_ESC_BEC: now also D2.2 (A); no longer D2.1 (K)
- net +5V_LOGIC: now also D1.1 (K), D2.1 (K); no longer D1.2 (A), D2.2 (A)
- net +5V_PM_BEC: now also D1.2 (A); no longer D1.1 (K)
- net GND: now also R30.2
- net MUX_SELECT: now also R30.1
Other:
- moved on the sheet: D1, D2
Changed lines of the file:
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@@
 		)
 	)
+	(label "MUX_SELECT"
+		(at 274.32 177.8 0)
+		(effects
+			(font
+				(size 1.016 1.016)
+			)
+			(justify right bottom)
+		)
+	)
+	(label "GND"
+		(at 274.32 185.42 0)
+		(effects
+			(font
+				(size 1.016 1.016)
+			)
+			(justify left bottom)
+		)
+	)
 	(label "ESP_SD_CS"
 		(at 172.72 49.53 0)
@@
 	(symbol
 		(lib_id "Device:R")
+		(at 274.32 181.61 0)
+		(unit 1)
+		(body_style 1)
+		(exclude_from_sim no)
+		(in_bom yes)
+		(on_board yes)
+		(in_pos_files yes)
+		(dnp no)
+		(property "Reference" "R30"
+			(at 274.32 177.8 0)
+			(show_name no)
+			(do_not_autoplace no)
+			(effects
+				(font
+					(size 1.27 1.27)
+				)
+			)
+		)
+		(property "Value" "10k"
+			(at 274.32 185.42 0)
+			(show_name no)
+			(do_not_autoplace no)
+			(effects
+				(font
+					(size 1.27 1.27)
+				)
+			)
+		)
+		(property "Footprint" "Resistor_SMD:R_0805_2012Metric_Pad1.20x1.40mm_HandSolder"
+			(at 274.32 181.61 0)
+			(hide yes)
+			(show_name no)
+			(do_not_autoplace no)
+			(effects
+				(font
+					(size 1.27 1.27)
+				)
+			)
+		)
+		(property "Datasheet" ""
+			(at 0 363.22 0)
+			(hide yes)
+			(show_name no)
+			(do_not_autoplace no)
+			(effects
+				(font
+					(size 1.27 1.27)
+				)
+			)
+		)
+		(property "Description" "MUX_SELECT fail-safe pull-down"
+			(at 274.32 181.61 0)
+			(show_name no)
+			(do_not_autoplace no)
+			(effects
+				(font
+					(size 1.27 1.27)
+				)
+			)
+		)
+		(pin "2"
+		)
+		(pin "1"
+		)
+		(instances
+			(project "FAST Controller"
+				(path "/3baf66a4-2d7e-4090-9aca-b1685f5554b9"
+					(reference "R30")
+					(unit 1)
+				)
+			)
+		)
+	)
+	(symbol
+		(lib_id "Device:R")
 		(at 175.26 198.12 0)
 		(unit 1)
@@
 	(symbol
 		(lib_id "Device:D_Schottky")
-		(at 63.5 228.6 0)
+		(at 63.5 228.6 180)
 		(unit 1)
 		(body_style 1)
@@
 	(symbol
 		(lib_id "Device:D_Schottky")
-		(at 99.06 228.6 0)
+		(at 99.06 228.6 180)
 		(unit 1)
 		(body_style 1)

Commit message: Update FAST Controller V2.2 schematic and ground stitching
Connections:
- net +5V_ESC_BEC: now also J10.2 (Pin_2), J11.2 (Pin_2), J12.2 (Pin_2), J13.2 (Pin_2), J14.2 (Pin_2), J15.2 (Pin_2), J8.2 (Pin_2), J9.2 (Pin_2); no longer J10.1 (Pin_1), J11.1 (Pin_1), J12.1 (Pin_1), J13.1 (Pin_1), J14.1 (Pin_1), J15.1 (Pin_1), J8.1 (Pin_1), J9.1 (Pin_1)
- net GND: now also J10.1 (Pin_1), J11.1 (Pin_1), J12.1 (Pin_1), J13.1 (Pin_1), J14.1 (Pin_1), J15.1 (Pin_1), J8.1 (Pin_1), J9.1 (Pin_1); no longer J10.2 (Pin_2), J11.2 (Pin_2), J12.2 (Pin_2), J13.2 (Pin_2), J14.2 (Pin_2), J15.2 (Pin_2), J8.2 (Pin_2), J9.2 (Pin_2)
Changed lines of the file:
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@@
 		)
 	)
-	(label "+5V_ESC_BEC"
+	(label "GND"
 		(at 350.52 226.06 0)
 		(effects
@@
 		)
 	)
-	(label "GND"
+	(label "+5V_ESC_BEC"
 		(at 350.52 228.6 0)
 		(effects
@@
 		)
 	)
-	(label "+5V_ESC_BEC"
+	(label "GND"
 		(at 294.64 223.52 0)
 		(effects
@@
 		)
 	)
-	(label "GND"
+	(label "+5V_ESC_BEC"
 		(at 294.64 226.06 0)
 		(effects
@@
 		)
 	)
-	(label "+5V_ESC_BEC"
+	(label "GND"
 		(at 294.64 240.03 0)
 		(effects
@@
 		)
 	)
-	(label "GND"
+	(label "+5V_ESC_BEC"
 		(at 350.52 245.11 0)
 		(effects
@@
 		)
 	)
-	(label "GND"
+	(label "+5V_ESC_BEC"
 		(at 294.64 209.55 0)
 		(effects
@@
 		)
 	)
-	(label "+5V_ESC_BEC"
+	(label "GND"
 		(at 350.52 242.57 0)
 		(effects
@@
 		)
 	)
-	(label "+5V_ESC_BEC"
+	(label "GND"
 		(at 294.64 190.5 0)
 		(effects
@@
 		)
 	)
-	(label "GND"
+	(label "+5V_ESC_BEC"
 		(at 350.52 212.09 0)
 		(effects
@@
 		)
 	)
-	(label "GND"
+	(label "+5V_ESC_BEC"
 		(at 350.52 195.58 0)
 		(effects
@@
 		)
 	)
-	(label "GND"
+	(label "+5V_ESC_BEC"
 		(at 294.64 242.57 0)
 		(effects
@@
 		)
 	)
-	(label "+5V_ESC_BEC"
+	(label "GND"
 		(at 350.52 209.55 0)
 		(effects
@@
 		)
 	)
-	(label "GND"
+	(label "+5V_ESC_BEC"
 		(at 294.64 193.04 0)
 		(effects
@@
 		)
 	)
-	(label "+5V_ESC_BEC"
+	(label "GND"
 		(at 294.64 207.01 0)
 		(effects
@@
 		)
 	)
-	(label "+5V_ESC_BEC"
+	(label "GND"
 		(at 350.52 193.04 0)
 		(effects
@@
 		(dnp no)
 		(property "Reference" "U1"
-			(at 62.23 63.5 0)
+			(at 59.69 45.72 0)
 			(show_name no)
 			(do_not_autoplace no)
@@
 		)
 		(property "Value" "FAST Teensy 4.0 DIP Carrier"
-			(at 62.23 71.12 0)
+			(at 59.69 88.9 0)
 			(show_name no)
 			(do_not_autoplace no)
